File: display_module/display_module.kicad_pcb (KiCad board)
At the start: 2 copper layers, 52 x 90 mm, 36 parts, among them J1 Conn_01x03_Female, J2 Conn_01x03_Male, J3 Conn_01x03_Female, J4 Conn_01x03_Male, J5 RESET, J6 HIGH, J7 PROG, J8 GND, SW1 PRIM, SW2 SEC, U1 74LS47, U2 74LS193, U3 MAN3410A, U4 74LS47, U5 74LS193, U6 MAN3410A

Commit message: Migrated to KiCad 6
Connections:
- net /IN_CLK renamed /CLK_{IN}
- U2 pad 12: (no net) -> unconnected-(U2-Pad12)
- U2 pad 13: (no net) -> unconnected-(U2-Pad13)
- U3 pad 12: (no net) -> unconnected-(U3-Pad12)
- U3 pad 4: (no net) -> unconnected-(U3-Pad4)
- U3 pad 5: (no net) -> unconnected-(U3-Pad5)
- U3 pad 6: (no net) -> unconnected-(U3-Pad6)
- U3 pad 9: (no net) -> unconnected-(U3-Pad9)
- U5 pad 12: (no net) -> unconnected-(U5-Pad12)
- U5 pad 13: (no net) -> unconnected-(U5-Pad13)
- U6 pad 12: (no net) -> unconnected-(U6-Pad12)
- U6 pad 4: (no net) -> unconnected-(U6-Pad4)
- U6 pad 5: (no net) -> unconnected-(U6-Pad5)
- U6 pad 6: (no net) -> unconnected-(U6-Pad6)
- U6 pad 9: (no net) -> unconnected-(U6-Pad9)
Other:
- net class Default removed
