File: display_module/display_module.kicad_pcb (KiCad board)
At the start: 2 copper layers, 52 x 90 mm, 36 parts, among them J1 Conn_01x03_Female, J2 Conn_01x03_Male, J3 Conn_01x03_Female, J4 Conn_01x03_Male, J5 RESET, J6 HIGH, J7 PROG, J8 GND, SW1 PRIM, SW2 SEC, U1 74LS47, U2 74LS193, U3 MAN3410A, U4 74LS47, U5 74LS193, U6 MAN3410A

Commit message: New schematics and minor rev for display
Added a signal name to the display board for the data load signals for each counter.
Connections:
- net Net-(R14-Pad1) renamed /~{LOAD}_{SEC}
- net Net-(R6-Pad1) renamed /~{LOAD}_{PRIM}
