File: reset_module/reset_modules.kicad_pcb (KiCad board)
At the start: 2 copper layers, 64.8 x 33 mm, 17 parts, among them J1 Conn_01x08_Female, J10 Conn_01x03_Male, J11 DISP, J12 Conn_01x03_Male, J13 Conn_01x03_Male, J14 Conn_01x03_Male, J15 Conn_01x03_Male, J2 Conn_01x08_Female, J3 Conn_01x04_Female, J4 Conn_01x04_Female, J5 Conn_01x03_Male, J6 Conn_01x03_Male, J7 Conn_01x03_Male, J8 Conn_01x03_Male, J9 Conn_01x03_Male, U1 74LS32, U2 74LS08

Commit message: Migrated to KiCad 6
Other:
- net class Default removed
