File: signal_generator/signal_generator.kicad_pcb (KiCad board)
At the start: 2 copper layers, 30 x 65.2 mm, 14 parts, among them J1 OUT, J2 OUT, J3 PWR, U1 CD4060, U2 CD4060, Y1 32768

Commit message: Migrated to KiCad 6
Other:
- net class Default removed
